File: CarteComm/Wifi/hardware/AIO_AGV_Control_V5.0.1/AIO_AGV_Control_V5.0.1.kicad_sch (KiCad schematic)
At the start: 0 parts

Commit message: docs(wifi): runbook de déploiement complet
DEPLOY.md : procédure opérationnelle en 11 phases, des mesures préalables au
procès-verbal de recette.

Trois points mis en tête parce qu'ils sont irréversibles ou bloquants :
- flasher détruit le firmware d'origine si la sauvegarde échoue — la phase 2
  donne les commandes esptool/avrdude, et impose une décision écrite du client
  si les bits de protection interdisent la relecture ;
- les niveaux du bus ne sont pas mesurés : la phase 1 est bloquante ;
- l'accord du service informatique est le chemin critique, à lancer le jour 1.

Contient aussi : configuration Mosquitto durcie avec ACL par topic (l'AGV ne
peut publier que sur ce qui le concerne), l'ordre de flash imposé (ATmega
d'abord, il démarre en safe_stop), dix essais de dégradation dont le
débranchement de la liaison inter-MCU en pleine course, un tableau de
diagnostic sur site et une fiche de recette à viser.

Co-Authored-By: Claude Opus 5 <noreply@anthropic.com>
Parts:
- added A1: Clone_Mega2560_Pro_Socket, arduino-library:Clone_Mega2560_Pro_Socket, symbol arduino-library:Clone_Mega2560_Pro_Socket
- added D1: D, Diode_THT:D_DO-41_SOD81_P10.16mm_Horizontal, symbol Device:D
- added R1: 1k, Resistor_THT:R_Axial_DIN0411_L9.9mm_D3.6mm_P12.70mm_Horizontal, symbol Device:R
- added T14: IRF520, IRF520:TO220BV, symbol IRF520:IRF520
- added U1: L7806, symbol Regulator_Linear:L7806
- added U2: ESP32-WROOM-32, RF_Module:ESP32-WROOM-32, symbol RF_Module:ESP32-WROOM-32
- added U3: TDN_5-2411WISM, Converter_DCDC:Converter_DCDC_TRACO_TDN_5-xxxxWISM_SMD, symbol Regulator_Switching:TDN_5-2411WISM
Connections:
- new net: A1.D48, R1.1, T14.G
- new net: U2.1 (GND), U2.15 (GND), U2.38 (GND), U2.39 (GND)
