File: CarteComm/Wifi/hardware/AIO_AGV_Control_V5.0.1/AIO_AGV_Control_V5.0.1.kicad_pcb (KiCad board)
At the start: 2 copper layers, 6 parts, among them T14 IRF520, U2 ESP32-WROOM-32, U3 TDN_5-2411WISM

Commit message: KiCad AGV Control 5.0.1
Parts:
- removed U2: ESP32-WROOM-32, RF_Module:ESP32-WROOM-32
- added J1: DB25_Pins, DB25P564CTXLF:AMPHENOL_DB25P564CTXLF, F.Cu at (192.8, 52.7)
- added J2: DB25_Socket, DB25S564GTLF:AMPHENOL_DB25S564GTLF, F.Cu at (175.3, 125.9)
- added LM1: L7806, L7806CV:TO255P1020X450X1968-3B, F.Cu at (127.0, 146.0)
- added R10: 1k, Resistor_THT:R_Axial_DIN0411_L9.9mm_D3.6mm_P12.70mm_Horizontal, F.Cu at (75.6, 51.2)
- added R11: 1k, Resistor_THT:R_Axial_DIN0411_L9.9mm_D3.6mm_P12.70mm_Horizontal, F.Cu at (75.8, 60.0)
- added R12: 1k, Resistor_THT:R_Axial_DIN0411_L9.9mm_D3.6mm_P12.70mm_Horizontal, F.Cu at (75.8, 69.0)
- added R14: 1k, Resistor_THT:R_Axial_DIN0411_L9.9mm_D3.6mm_P12.70mm_Horizontal, F.Cu at (125.5, 42.0)
- added R15: 1k, Resistor_THT:R_Axial_DIN0411_L9.9mm_D3.6mm_P12.70mm_Horizontal, F.Cu at (125.3, 51.0)
- added R16: 1k, Resistor_THT:R_Axial_DIN0411_L9.9mm_D3.6mm_P12.70mm_Horizontal, F.Cu at (125.8, 60.0)
- added R17: 1k, Resistor_THT:R_Axial_DIN0411_L9.9mm_D3.6mm_P12.70mm_Horizontal, F.Cu at (125.5, 69.0)
- added R18: 1k, Resistor_THT:R_Axial_DIN0411_L9.9mm_D3.6mm_P12.70mm_Horizontal, F.Cu at (92.4, 42.0)
- added R19: 1k, Resistor_THT:R_Axial_DIN0411_L9.9mm_D3.6mm_P12.70mm_Horizontal, F.Cu at (92.2, 51.2)
- added R2: 1k, Resistor_THT:R_Axial_DIN0411_L9.9mm_D3.6mm_P12.70mm_Horizontal, F.Cu at (58.9, 51.2)
- added R20: 1k, Resistor_THT:R_Axial_DIN0411_L9.9mm_D3.6mm_P12.70mm_Horizontal, F.Cu at (92.5, 60.0)
- added R21: 1k, Resistor_THT:R_Axial_DIN0411_L9.9mm_D3.6mm_P12.70mm_Horizontal, F.Cu at (92.3, 69.0)
- added R22: 1k, Resistor_THT:R_Axial_DIN0411_L9.9mm_D3.6mm_P12.70mm_Horizontal, F.Cu at (142.1, 42.0)
- added R23: 1k, Resistor_THT:R_Axial_DIN0411_L9.9mm_D3.6mm_P12.70mm_Horizontal, F.Cu at (141.9, 51.0)
- added R24: 1k, Resistor_THT:R_Axial_DIN0411_L9.9mm_D3.6mm_P12.70mm_Horizontal, F.Cu at (142.4, 60.0)
- added R3: 1k, Resistor_THT:R_Axial_DIN0411_L9.9mm_D3.6mm_P12.70mm_Horizontal, F.Cu at (59.1, 60.0)
- added R30: 4.7k, Resistor_THT:R_Axial_DIN0411_L9.9mm_D3.6mm_P12.70mm_Horizontal, F.Cu at (69.8, 122.5)
- added R31: 2.2k, Resistor_THT:R_Axial_DIN0411_L9.9mm_D3.6mm_P12.70mm_Horizontal, F.Cu at (69.5, 139.2)
- added R4: 1k, Resistor_THT:R_Axial_DIN0411_L9.9mm_D3.6mm_P12.70mm_Horizontal, F.Cu at (59.1, 69.0)
- added R40: 22k, Resistor_THT:R_Axial_DIN0411_L9.9mm_D3.6mm_P12.70mm_Horizontal, F.Cu at (112.3, 142.0)
- added R41: 220k, Resistor_THT:R_Axial_DIN0411_L9.9mm_D3.6mm_P12.70mm_Horizontal, F.Cu at (112.5, 158.3)
- added R5: 1k, Resistor_THT:R_Axial_DIN0411_L9.9mm_D3.6mm_P12.70mm_Horizontal, F.Cu at (108.8, 42.0)
- added R6: 1k, Resistor_THT:R_Axial_DIN0411_L9.9mm_D3.6mm_P12.70mm_Horizontal, F.Cu at (108.7, 51.0)
- added R7: 1k, Resistor_THT:R_Axial_DIN0411_L9.9mm_D3.6mm_P12.70mm_Horizontal, F.Cu at (109.2, 60.0)
- added R8: 1k, Resistor_THT:R_Axial_DIN0411_L9.9mm_D3.6mm_P12.70mm_Horizontal, F.Cu at (108.8, 69.0)
- added R9: 1k, Resistor_THT:R_Axial_DIN0411_L9.9mm_D3.6mm_P12.70mm_Horizontal, F.Cu at (75.7, 42.0)
- added T1: IRF520, IRF520:TO220BV, F.Cu at (162.7, 63.4)
- added T10: IRF520, IRF520:TO220BV, F.Cu at (81.7, 44.5)
- added T11: IRF520, IRF520:TO220BV, F.Cu at (81.8, 53.5)
- added T12: IRF520, IRF520:TO220BV, F.Cu at (81.8, 62.5)
- added T15: IRF520, IRF520:TO220BV, F.Cu at (131.5, 44.5)
- added T16: IRF520, IRF520:TO220BV, F.Cu at (132.0, 53.5)
- added T17: IRF520, IRF520:TO220BV, F.Cu at (132.0, 62.5)
- added T18: IRF520, IRF520:TO220BV, F.Cu at (99.0, 35.5)
- added T19: IRF520, IRF520:TO220BV, F.Cu at (98.5, 44.5)
- added T2: IRF520, IRF520:TO220BV, F.Cu at (65.5, 44.5)
- added T20: IRF520, IRF520:TO220BV, F.Cu at (98.5, 53.5)
- added T21: IRF520, IRF520:TO220BV, F.Cu at (98.5, 62.5)
- added T22: IRF520, IRF520:TO220BV, F.Cu at (148.5, 35.5)
- added T23: IRF520, IRF520:TO220BV, F.Cu at (148.5, 44.5)
- added T24: IRF520, IRF520:TO220BV, F.Cu at (148.5, 53.5)
- added T3: IRF520, IRF520:TO220BV, F.Cu at (65.5, 53.5)
- added T4: IRF520, IRF520:TO220BV, F.Cu at (65.5, 62.5)
- added T5: IRF520, IRF520:TO220BV, F.Cu at (115.0, 35.5)
- added T6: IRF520, IRF520:TO220BV, F.Cu at (115.0, 44.5)
- added T7: IRF520, IRF520:TO220BV, F.Cu at (115.5, 53.5)
- added T8: IRF520, IRF520:TO220BV, F.Cu at (115.0, 62.5)
- added T9: IRF520, IRF520:TO220BV, F.Cu at (82.0, 35.5)
- added U1: ESP32-DEVKITC, ESP32-DEVKITC:MODULE_ESP32-DEVKITC, F.Cu at (66.7, 112.2)
- A1: footprint arduino-library:Arduino_Mega2560_R3_Shield -> arduino-library:Clone_Mega2560_Pro_Socket
- R1: footprint Resistor_THT:R_Axial_DIN0411_L9.9mm_D3.6mm_P20.32mm_Horizontal -> Resistor_THT:R_Axial_DIN0411_L9.9mm_D3.6mm_P12.70mm_Horizontal
- moved R1 98.3 mm to (156.3, 70.0)
- moved T14 93.8 mm to (132.0, 35.5)
- moved TDN1 73.5 mm to (101.8, 161.5), turned to -90 degrees
- moved D1 72.8 mm to (150.6, 112.0), turned to 180 degrees
- moved A1 29.4 mm to (88.2, 139.4), turned to 90 degrees
- renumbered U3 to TDN1
Connections:
- A1 pad A0: unconnected-(A1-PadA0) -> Net-(A1-PadA0)
- A1 pad A1: unconnected-(A1-PadA1) -> Net-(J2-P20)
- A1 pad A2: unconnected-(A1-PadA2) -> Net-(J2-P21)
- A1 pad A3: unconnected-(A1-PadA3) -> Net-(J2-P22)
- A1 pad A4: unconnected-(A1-PadA4) -> Net-(J2-P23)
- A1 pad A5: unconnected-(A1-PadA5) -> Net-(J2-P24)
- A1 pad D10: unconnected-(A1-PadD10) -> Net-(A1-PadD10)
- A1 pad D11: unconnected-(A1-PadD11) -> Net-(D1-A)
- A1 pad D12: unconnected-(A1-PadD12) -> Net-(A1-PadD12)
- A1 pad D15: unconnected-(A1-D15/RX3-PadD15) -> Net-(A1-D15/RX3)
- A1 pad D17: unconnected-(A1-D17/RX2-PadD17) -> Net-(A1-D17/RX2)
- A1 pad D19: unconnected-(A1-D19/RX1-PadD19) -> Net-(A1-D19/RX1)
- A1 pad D2: unconnected-(A1-D2_INT0-PadD2) -> Net-(A1-D2_INT0)
- A1 pad D21: unconnected-(A1-D21/SCL-PadD21) -> Net-(A1-D21/SCL)
- A1 pad D22: unconnected-(A1-PadD22) -> Net-(A1-PadD22)
- A1 pad D23: unconnected-(A1-PadD23) -> Net-(J2-P19)
- A1 pad D24: unconnected-(A1-PadD24) -> Net-(A1-PadD24)
- A1 pad D25: unconnected-(A1-PadD25) -> Net-(A1-PadD25)
- A1 pad D26: unconnected-(A1-PadD26) -> Net-(A1-PadD26)
- A1 pad D27: unconnected-(A1-PadD27) -> Net-(A1-PadD27)
- A1 pad D28: unconnected-(A1-PadD28) -> Net-(A1-PadD28)
- A1 pad D29: unconnected-(A1-PadD29) -> Net-(A1-PadD29)
- A1 pad D3: unconnected-(A1-D3_INT1-PadD3) -> Net-(A1-D3_INT1)
- A1 pad D30: unconnected-(A1-PadD30) -> Net-(A1-PadD30)
- A1 pad D31: unconnected-(A1-PadD31) -> Net-(A1-PadD31)
- A1 pad D33: unconnected-(A1-PadD33) -> Net-(A1-PadD33)
- A1 pad D35: unconnected-(A1-PadD35) -> Net-(A1-PadD35)
- A1 pad D37: unconnected-(A1-PadD37) -> Net-(A1-PadD37)
- A1 pad D39: unconnected-(A1-PadD39) -> Net-(A1-PadD39)
- A1 pad D4: unconnected-(A1-PadD4) -> Net-(A1-PadD4)
- A1 pad D41: unconnected-(A1-PadD41) -> Net-(A1-PadD41)
- A1 pad D43: unconnected-(A1-PadD43) -> Net-(A1-PadD43)
- A1 pad D44: unconnected-(A1-PadD44) -> Net-(A1-PadD44)
- A1 pad D45: unconnected-(A1-PadD45) -> Net-(A1-PadD45)
- A1 pad D46: unconnected-(A1-PadD46) -> Net-(A1-PadD46)
- A1 pad D47: unconnected-(A1-PadD47) -> Net-(A1-PadD47)
- A1 pad D49: unconnected-(A1-PadD49) -> Net-(A1-PadD49)
- A1 pad D5: unconnected-(A1-PadD5) -> Net-(A1-PadD5)
- A1 pad D50: unconnected-(A1-D50_MISO-PadD50) -> Net-(A1-D50_MISO)
- A1 pad D51: unconnected-(A1-D51_MOSI-PadD51) -> Net-(A1-D51_MOSI)
- A1 pad D52: unconnected-(A1-D52_SCK-PadD52) -> Net-(A1-D52_SCK)
- A1 pad D53: unconnected-(A1-D53_CS-PadD53) -> Net-(A1-D53_CS)
- A1 pad D6: unconnected-(A1-PadD6) -> Net-(A1-PadD6)
- A1 pad D7: unconnected-(A1-PadD7) -> Net-(A1-PadD7)
- A1 pad D8: unconnected-(A1-PadD8) -> Net-(A1-PadD8)
- A1 pad D9: unconnected-(A1-PadD9) -> Net-(A1-PadD9)
- A1 pad GND1: unconnected-(A1-GND-PadGND1) -> Net-(TDN1--VIN)
- A1 pad GND2: unconnected-(A1-GND-PadGND2) -> Net-(LM1-GND)
- D1 pad 1: unconnected-(D1-K-Pad1) -> Net-(D1-K)
- D1 pad 2: unconnected-(D1-A-Pad2) -> Net-(D1-A)
- R1 pad 1: Net-(A1-PadD48) -> Net-(A1-PadD27)
- R1 pad 2: unconnected-(R1-Pad2) -> Net-(J1-P25)
- T14 pad D: unconnected-(T14-PadD) -> Net-(J1-P14)
- T14 pad S: unconnected-(T14-PadS) -> Net-(J1-P25)
- TDN1 pad 1: unconnected-(U3-+VIN-Pad1) -> Net-(J2-P25)
- TDN1 pad 2: unconnected-(U3--VIN-Pad2) -> Net-(TDN1--VIN)
- TDN1 pad 4: unconnected-(U3-ON/OFF-Pad4) -> Net-(TDN1--VIN)
- TDN1 pad 6: unconnected-(U3--VOUT-Pad6) -> Net-(TDN1--VOUT)
- TDN1 pad 7: unconnected-(U3-+VOUT-Pad7) -> Net-(TDN1-+VOUT)
Routing:
- net Net-(J2-P25): track 0.00 -> 77.2 mm
- net Net-(A1-PadD10): track 0.00 -> 76.8 mm
- net Net-(J2-P19): track 0.00 -> 74.6 mm
- net Net-(A1-PadD8): track 0.00 -> 71.3 mm
- net Net-(A1-PadD12): track 0.00 -> 70.4 mm
- net Net-(A1-D21/SCL): track 0.00 -> 70.1 mm
- net Net-(TDN1--VOUT): track 0.00 -> 67.7 mm
- net Net-(A1-PadD6): track 0.00 -> 65.8 mm
- net Net-(A1-D19/RX1): track 0.00 -> 65.6 mm
- net Net-(A1-D53_CS): track 0.00 -> 64.8 mm
- net Net-(A1-D17/RX2): track 0.00 -> 61.2 mm
- net Net-(A1-PadD4): track 0.00 -> 60.3 mm
- net Net-(A1-D15/RX3): track 0.00 -> 54.7 mm
- net Net-(TDN1-+VOUT): track 0.00 -> 54.4 mm
- net Net-(A1-D2_INT0): track 0.00 -> 54.1 mm
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
Commit message: Update routage PCB
Parts:
- moved T24 100.7 mm to (48.0, 47.3), turned to 90 degrees
- moved J1 96.1 mm to (98.9, 31.7), turned to 180 degrees
- moved T23 91.5 mm to (57.0, 47.3), turned to 90 degrees
- moved R24 88.2 mm to (54.5, 53.9), turned to 90 degrees
- moved R2 84.1 mm to (141.0, 69.3), turned to 90 degrees
- moved T22 83.4 mm to (66.0, 47.5), turned to 90 degrees
- moved R23 78.5 mm to (63.5, 53.9), turned to 90 degrees
- moved R3 73.5 mm to (132.0, 69.3), turned to 90 degrees
- moved T2 71.2 mm to (134.3, 62.8), turned to 90 degrees
- moved R22 70.6 mm to (72.5, 53.9), turned to 90 degrees
- moved R4 63.9 mm to (123.0, 69.3), turned to 90 degrees
- moved T3 60.8 mm to (125.5, 63.0), turned to 90 degrees
- moved T4 51.0 mm to (116.5, 62.5), turned to 90 degrees
- moved T12 38.3 mm to (43.5, 63.5), turned to 90 degrees
- moved T8 35.1 mm to (80.0, 62.9), turned to 90 degrees
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Connections:
- R11 pad 1: unconnected-(R11-Pad1) -> Net-(A1-PadD33)
- T9 pad D: Net-(J1-P25) -> Net-(J1-Pad9)
Routing:
- net Net-(J1-P25): track 3.11 -> 403.2 mm
- net Net-(A1-PadD43): track 0.00 -> 131.2 mm
- net Net-(A1-D50_MISO): track 0.00 -> 95.6 mm
- net Net-(A1-PadD25): track 0.00 -> 89.9 mm
- net Net-(J2-P24): track 0.00 -> 88.4 mm
- net Net-(A1-PadD26): track 0.00 -> 86.9 mm
- net Net-(A1-PadD48): track 0.00 -> 84.7 mm
- net Net-(A1-PadD31): track 0.00 -> 83.4 mm
- net Net-(J2-P22): track 0.00 -> 82.4 mm
- net Net-(J2-P23): track 0.00 -> 82.1 mm
- net Net-(A1-PadD22): track 0.00 -> 82.0 mm
- net Net-(A1-D51_MOSI): track 0.00 -> 76.8 mm
- net Net-(J2-P21): track 0.00 -> 73.7 mm
- net Net-(A1-PadD49): track 0.00 -> 73.7 mm
- net Net-(J2-P20): track 0.00 -> 69.6 mm
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