File: CarteComm/Wifi/hardware/AIO_AGV_Control_V6.0/AIO_AGV_Control_V6.0.kicad_pcb (KiCad board)
At the start: 2 copper layers, 57 parts, among them J1 DB25_Pins, J2 DB25_Socket, T1 IRF520, T10 IRF520, T11 IRF520, T12 IRF520, T14 IRF520, T15 IRF520, T16 IRF520, T17 IRF520, T18 IRF520, T19 IRF520, T2 IRF520, T20 IRF520, T21 IRF520, T22 IRF520, T23 IRF520, T24 IRF520, T3 IRF520, T4 IRF520, T5 IRF520, T6 IRF520, T7 IRF520, T8 IRF520, T9 IRF520, U1 ESP32-DEVKITC

Commit message: feat(bom): resserrer les nomenclatures sur les composants déterminants
Les accessoires arbitrables selon le budget - antennes, boîtiers, coffrets,
enveloppes murales, câbles, plaques gravées - sortent de l'affichage et des
sous-totaux. Trente-six lignes qui se substituent librement d'un fournisseur à
l'autre et n'engagent aucun choix de conception : elles allongeaient la lecture
sans rien apporter à la décision.

Elles restent définies dans generer_bom.py, marquées core=False. Rien n'est
perdu, et un accessoire redevient visible en changeant un mot.

Chaque BOM s'ouvre désormais sur un bloc Total, par variante, avec une colonne
rappelant le montant des accessoires écartés. Sans ce rappel, un total amputé
des antennes et des boîtiers se lirait comme un coût d'achat complet.

Deux effets de bord traités plutôt que laissés passer. Le point de bascule
A1/A3 se calculait sur des boutons dont le prix tient justement au boîtier IP65
et au poussoir Ø22 : retirer ces lignes inversait le classement. Ce tableau
raisonne donc accessoires compris, le dit, et le point de bascule est maintenant
CALCULÉ au lieu d'être asséné - il passe de 8 à 9 stations. Deux coûts par
station encore codés en dur à 50 EUR ont été branchés sur les sections.

README.md et COMPARAISON.md gardent la base complète, pour la même raison :
comparer des architectures sans leurs boîtiers fausserait le classement. Leurs
chiffres sont plus élevés que ceux des BOM, et les deux documents le disent.
Deux totaux LoRa y étaient restés périmés depuis la réutilisation de la carte
V5.0.1 - corrigés à 208 et 307 EUR.

Contrôle : core + accessoires retombe exactement sur les six totaux complets
cités par les documents de comparaison.

Co-Authored-By: Claude Opus 5 <noreply@anthropic.com>
Parts:
- added U2: RFM95W-868S2, RF_Module:HOPERF_RFM9XW_SMD, F.Cu at (40.0, 100.0)
Connections:
- U1 pad 1: unconnected-(U1-3V3-Pad1) -> Net-(U1-3V3)
- U1 pad 10: unconnected-(U1-IO26-Pad10) -> Net-(U1-IO26)
- U1 pad 29: unconnected-(U1-IO5-Pad29) -> Net-(U1-IO5)
- U1 pad 30: unconnected-(U1-IO18-Pad30) -> Net-(U1-IO18)
- U1 pad 31: unconnected-(U1-IO19-Pad31) -> Net-(U1-IO19)
- U1 pad 37: unconnected-(U1-IO23-Pad37) -> Net-(U1-IO23)
- U1 pad 38: unconnected-(U1-GND3-Pad38) -> Net-(U1-GND3)
Routing:
- net Net-(U1-GND3): track 0.00 -> 109.5 mm
- net Net-(U1-IO23): track 0.00 -> 96.0 mm
- net Net-(J1-P25): track 403.2 -> 475.2 mm
- net Net-(U1-IO5): track 0.00 -> 48.9 mm
- net Net-(U1-IO18): track 0.00 -> 46.0 mm
- net Net-(J1-Pad3): track 0.00 -> 45.4 mm
- net Net-(J1-Pad4): track 0.00 -> 37.9 mm
- net Net-(J1-Pad5): track 0.00 -> 34.3 mm
- net Net-(U1-IO19): track 0.00 -> 32.7 mm
- net Net-(J1-Pad6): track 0.00 -> 31.9 mm
- net Net-(U1-3V3): track 0.00 -> 26.4 mm
- net Net-(U1-IO26): track 0.00 -> 25.3 mm
- net Net-(J2-P20): track 69.6 -> 74.2 mm
- net Net-(J2-P21): track 73.7 -> 77.4 mm
- net Net-(A1-PadD10): track 59.3 -> 56.1 mm
